Commit message: Revert "Complete World with updated Deuterium Model"

File: src/hydrogen/model/main_frame.xacro (robot description, xacro)
@@ -5,13 +5,18 @@
     <link name="hydrogen_frame">
       <inertial>
-        <origin xyz="0.0 0.0 0.0" rpy="0 0 0"/>
-        <mass value="12.0"/>
-<inertia ixx="0.391803" iyy="0.876695" izz="1.065444" ixy="0.0" iyz="0.0" ixz="-0.006759"/>
+        <origin xyz="0.0 0.0 -0.25" rpy="0 0 0"/>
+        <mass value="40.0"/>
+        <inertia
+          ixx="0.2276"
+          ixy="-0.004544"
+          ixz="-0.0004496"
+          iyy="0.1921"
+          iyz="-0.0001196"
+          izz="0.3559"/>
       </inertial>
       <visual>
-      <origin xyz="0.008 0.0 0.0" rpy="0 0 1.57"/>
         <geometry>
           <mesh
-            filename="file://$(find hydrogen)/meshes/auv.stl"
+            filename="file://$(find hydrogen)/meshes/auv2.stl"
             scale="0.001 0.001 0.001"/>
         </geometry>
@@ -21,7 +26,7 @@
       </visual>
       <collision name="hydrogen_frame_collision">
-        <origin xyz="0.0 0.0 0.1" rpy="0 0 0"/>
+        <origin xyz="0.008 0.0 0.0" rpy="0 0 0"/>
         <geometry>
-          <box size="0.75 0.55 0.3"/>
+          <box size="0.45 0.45 0.25"/>
         </geometry>
       </collision>

File: src/hydrogen/model/propellers.xacro (robot description, xacro)
@@ -75,32 +75,32 @@
       izz="0.0008"/>
     <!-- Joints -->
-    <joint name="back_propeller_joint" type="continuous">
+    <joint name="front_propeller_joint" type="continuous">
       <parent link="hydrogen_frame"/>
       <child link="front_propeller"/>
-      <origin xyz="-0.3219 -0 0.0775" rpy="0 0 0"/>
+      <origin xyz="-0.223 -0.00725 0.002" rpy="0 0 0"/>
+      <axis xyz="0 0 1"/>
+    </joint>
+    <joint name="left_propeller_1_joint" type="continuous">
+      <parent link="hydrogen_frame"/>
+      <child link="left_propeller_1"/>
+      <origin xyz="-0.0631 -0.1734 0.016" rpy="-1.57 0 1.57"/>
+      <axis xyz="0 0 1"/>
+    </joint>
+    <joint name="left_propeller_2_joint" type="continuous">
+      <parent link="hydrogen_frame"/>
+      <child link="left_propeller_2"/>
+      <origin xyz="0.0697 -0.1734 0.002" rpy="0 0 0"/>
       <axis xyz="0 0 1"/>
     </joint>
     <joint name="right_propeller_1_joint" type="continuous">
       <parent link="hydrogen_frame"/>
-      <child link="left_propeller_1"/>
-      <origin xyz="-0.1532 0.222 0.085" rpy="-1.57 0 1.57"/>
+      <child link="right_propeller_1"/>
+      <origin xyz="-0.0631 0.1734 0.016" rpy="-1.57 0 1.57"/>
       <axis xyz="0 0 1"/>
     </joint>
     <joint name="right_propeller_2_joint" type="continuous">
       <parent link="hydrogen_frame"/>
-      <child link="left_propeller_2"/>
-      <origin xyz="0.1737 0.222 0.0775" rpy="0 0 0"/>
-      <axis xyz="0 0 1"/>
-    </joint>
-    <joint name="left_propeller_1_joint" type="continuous">
-      <parent link="hydrogen_frame"/>
-      <child link="right_propeller_1"/>
-      <origin xyz="-0.1532 -0.222 0.085" rpy="-1.57 0 1.57"/>
-      <axis xyz="0 0 1"/>
-    </joint>
-    <joint name="left_propeller_2_joint" type="continuous">
-      <parent link="hydrogen_frame"/>
       <child link="right_propeller_2"/>
-      <origin xyz="00.1737 -0.222 0.0775" rpy="0 0 0"/>
+      <origin xyz="0.0697 0.1734 0.002" rpy="0 0 0"/>
       <axis xyz="0 0 1"/>
     </joint>

File: src/hydrogen/model/robot.xacro (robot description, xacro)
@@ -10,10 +10,10 @@
     name="zed_camera_front_link"
     parent="hydrogen_frame"
-    xyz="0.31 0 0.1"
+    xyz="0.162 0 0.016"
     rpy="0 0 0"/>
   <xacro:zed_camera
     name="zed_camera_down_link"
     parent="hydrogen_frame"
-    xyz="0.17 0 -0.04"
+    xyz="0.05 0 -0.08"
     rpy="0 1.5708 0"/>
 </robot>

Commit message: added teleop nodes (still under testing)

File: src/hydrogen/model/main_frame.xacro (robot description, xacro)
@@ -6,5 +6,5 @@
       <inertial>
         <origin xyz="0.0 0.0 0.0" rpy="0 0 0"/>
-        <mass value="45.0"/>
+        <mass value="96.0"/>
         <inertia
           ixx="0.2276"
